File: PCB/randir/_autosave-randir.kicad_pcb (KiCad board)
At the start: 2 copper layers, 136.7 x 59.6 mm, 29 parts, among them SW1 SW_Push, SW10 SW_Push, SW2 SW_Push, SW3 SW_Push, SW4 SW_Push, SW5 SW_Push, SW7 SW_Push, SW8 SW_Push, SW9 SW_Push, U1 nice_nano_Toby

Commit message: js
Parts:
- removed the ? at (148.3, 79.6)
- moved SW10 17.0 mm to (162.5, 77.4), turned to 180 degrees
- moved SW5 17.0 mm to (179.5, 77.4), turned to 180 degrees
Routing:
- net GND: track 23.0 -> 40.4 mm
- net Bat+: track 4.07 -> 8.14 mm
Other:
- outline, holes or cut-outs redrawn

Commit message: dgf
Parts:
- removed the ? at (167.7, 106.0)
- added REF**: toby_slide_in, footprints3:toby_slide_in, F.Cu at (144.5, 76.9)
- added REF**: toby_slide_in, footprints3:toby_slide_in, F.Cu at (139.5, 66.9)
- added REF**: toby_slide_in, footprints3:toby_slide_in, F.Cu at (144.5, 66.9)
- added REF**: toby_slide_in, footprints3:toby_slide_in, F.Cu at (154.5, 66.9)
- added REF**: toby_slide_down, footprints3:toby_slide_down, F.Cu at (244.1, 108.0)
- moved REF** 82.4 mm to (42.6, 93.4)
Other:
- outline, holes or cut-outs redrawn
