File: PCB/randir/randir.kicad_pcb (KiCad board)
At the start: 2 copper layers, 136.7 x 59.6 mm, 29 parts, among them SW1 SW_Push, SW10 SW_Push, SW2 SW_Push, SW3 SW_Push, SW4 SW_Push, SW5 SW_Push, SW7 SW_Push, SW8 SW_Push, SW9 SW_Push, U1 nice_nano_Toby

Commit message: sides
Parts:
- removed ? (x10): , 
- removed ENC1 (x2): toby_enc, PCM_Switch_Keyboard_Hotswap_Kailh:toby_enc
- removed the REF** at (65.5, 14.2)
- removed the REF** at (114.4, 105.7)
- removed the REF** at (74.4, 88.7)
- removed TJS1: thumbstick1, PCM_Switch_Keyboard_Hotswap_Kailh:toby_js
- added REF**: ANO-Toby-revers, ANO-reversible:ANO-Toby-revers, F.Cu at (118.0, 110.5)
- moved REF** 65.7 mm to (118.5, 50.0), turned to -92 degrees
- moved REF** 58.3 mm to (118.2, 57.6), turned to 88 degrees
- moved SW10 53.4 mm to (126.1, 75.5), turned to -92 degrees
- moved SW1 29.9 mm to (51.9, 115.0), turned to -30 degrees
- moved SW1 29.6 mm to (37.2, 106.5), turned to -30 degrees
- moved SW7 29.2 mm to (68.2, 95.8), turned to 34 degrees
- moved SW8 28.8 mm to (82.0, 84.1), turned to 34 degrees
- moved SW2 28.7 mm to (58.7, 81.7), turned to 34 degrees
- moved SW9 28.7 mm to (101.2, 79.3), turned to 24 degrees
- moved SW3 28.3 mm to (72.5, 70.0), turned to 34 degrees
- moved SW4 28.1 mm to (94.3, 63.8), turned to 24 degrees
- moved SW5 15.5 mm to (147.5, 81.0), turned to -2 degrees
- moved U1 13.8 mm to (156.2, 67.3), turned to 88 degrees
Connections:
- SW1 pad 1: (no net) -> D9
- SW1 pad 2: (no net) -> GND (x2)
- SW1 pad 1: (no net) -> D16
- SW10 pad 1: (no net) -> D0
- SW10 pad 2: (no net) -> GND
- SW2 pad 1: (no net) -> D8
- SW2 pad 2: (no net) -> GND
- SW3 pad 1: (no net) -> D7
- SW3 pad 2: (no net) -> GND
- SW4 pad 1: (no net) -> D6
- SW4 pad 2: (no net) -> GND
- SW5 pad 1: (no net) -> D1
- SW5 pad 2: (no net) -> GND
- SW7 pad 1: (no net) -> D14
- SW7 pad 2: (no net) -> GND
- SW8 pad 1: (no net) -> D15
- SW8 pad 2: (no net) -> GND
- SW9 pad 1: (no net) -> D18
- SW9 pad 2: (no net) -> GND
- U1 pad 0: (no net) -> D0
- U1 pad 1: (no net) -> D1
- U1 pad 10: (no net) -> D10
- U1 pad 14: (no net) -> D14
- U1 pad 15: (no net) -> D15
- U1 pad 16: (no net) -> D16
- U1 pad 18: (no net) -> D18
- U1 pad 19: (no net) -> D19
- U1 pad 2: (no net) -> D2
- U1 pad 20: JS_Y -> D20
- U1 pad 21: JS_X -> D21
- U1 pad 3: (no net) -> D3
- U1 pad 4: (no net) -> D4
- U1 pad 5: (no net) -> D5
- U1 pad 6: (no net) -> D6
- U1 pad 7: (no net) -> D7
- U1 pad 8: (no net) -> D8
- U1 pad 9: (no net) -> D9
Routing:
- net GND: track 23.0 -> 582.8 mm, vias 0 -> 1
- net D16: track 0.00 -> 156.9 mm
- net D9: track 0.00 -> 138.3 mm
- net D14: track 0.00 -> 127.9 mm
- net D15: track 0.00 -> 110.2 mm
- net D8: track 0.00 -> 109.8 mm
- net D4: track 0.00 -> 105.3 mm
- net D7: track 0.00 -> 96.5 mm
- net D2: track 0.00 -> 94.5 mm
- net D18: track 0.00 -> 89.3 mm
- net D5: track 0.00 -> 87.7 mm
- net D20: track 0.00 -> 83.2 mm
- net D21: track 0.00 -> 77.5 mm
- net D6: track 0.00 -> 75.4 mm
- net D3: track 0.00 -> 72.9 mm
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Other:
- board size 136.7 x 59.6 mm -> 135.3 x 84.3 mm
- board text added: "0431 933 944"
- board text added: "Developed by Toby Price"
- board text added: "If lost, please return"
- board text added: "Randir Keyboard (v2)"
- board text added: "face down"
